Commit message: fix trajectory execution, the end effector pointing inward

File: src/aubo_description/urdf/aubo_i3.urdf (robot description, URDF)
Before this commit: robot aubo_i3, 8 links, 7 joints
Links:
- added link tool_link; visual cylinder length=0.04 radius=0.005
Joints:
- added joint tool_joint: type fixed, parent wrist3_Link, child tool_link, origin xyz=0 0 0 rpy=0 1.5708 0
